File: Electronics/Medium_Power_switch/Medium_switch_1.sch (EAGLE design)
At the start: 37 parts, among them U1 BTS700151ESPXUMA1, U2 AP63205WU-7

Commit message: Nuevos esquematicos y PCB
Parts:
- added D1, D3: (no value), diode:DIODE-MICROMELF-R
- D2: device diode:DIODE-MICROMELF-R -> diode:DIODE-MINIMELF
- RBAT1, RESV+: value (none) -> 23k
- RBAT2, RBAT4, RBAT5, RCH2: value (none) -> 10k
- RBAT3, RCH1, RDIAGEN, RPWREN: value (none) -> 1.2k
Connections:
- net BOTON: now also D3.C
- net GND: now also D1.A, D3.A
- net N$11: now also D1.C
